Commit message: Contact points for a mug and a mug tree. Visualizer.

File: data/mug_trees/mug_tree.urdf (robot description, URDF)
Before this commit: robot mug.urdf, 3 links, 2 joints
Links:
- removed link ap2
- link ap1: geometry visual sphere radius=0.005
- link base: geometry collision mesh filename=mug_tree_convex.obj scale=0.004 0.004 0.004; visual mesh filename=mug_tree.stl scale=0.004 0.004 0.004
Joints:
- removed joint base_to_ap2
- joint base_to_ap1: origin xyz=0 0.048 0.107 -> xyz=0.028 0.05 0.105
