Commit message: collision detection; clone picks and places

File: data/mug_tree/mug_tree.urdf (robot description, URDF)
Before this commit: robot mug_tree.urdf, 2 links, 1 joints
Links:
- removed link ap1
- link base: geometry collision mesh filename=mug_tree_convex.obj scale=0.01 0.01 0.01; visual mesh filename=mug_tree.stl scale=0.01 0.01 0.01
Joints:
- removed joint base_to_ap1

File: data/mugs/0.urdf (robot description, URDF)
Before this commit: robot mug.urdf, 3 links, 2 joints
Links:
- removed link ap1
- removed link ap2
- link base: geometry collision mesh filename=0_convex.obj scale=1 1 1; visual mesh filename=0_convex.obj scale=1 1 1
Joints:
- removed joint base_to_ap1
- removed joint base_to_ap2
