Commit message: Progress on getting a collision free path to the tree.

File: data/mugs/test/0.urdf (robot description, URDF)
Before this commit: robot mug.urdf, 1 links, 0 joints
Links:
- link baseLink: geometry collision mesh filename=0_convex.obj scale=1 1 1; visual mesh filename=0_convex.obj scale=1 1 1

File: data/simple_trees/test/0.urdf (robot description, URDF)
Before this commit: robot tree.urdf, 1 links, 0 joints
Links:
- link baseLink: geometry collision mesh filename=0_convex.obj scale=1 1 1; visual mesh filename=0_convex.obj scale=1 1 1

Commit message: New mugs and trees. Workspace is set up. Cloning works without motion planning.

File: data/mugs/test/0.urdf (robot description, URDF)
Before this commit: robot mug.urdf, 1 links, 0 joints
Links:
- link baseLink: geometry collision mesh filename=0_convex.obj scale=1 1 1; visual mesh filename=0.stl scale=1 1 1

File: data/simple_trees/test/0.urdf (robot description, URDF)
Before this commit: robot tree.urdf, 1 links, 0 joints
Links:
- link baseLink: geometry collision mesh filename=0_convex.obj scale=1 1 1; visual mesh filename=0.stl scale=1 1 1
