Commit message: Refactored and fixed demonstration recording. Augmented the visualization of placement warping.

File: data/real_tree.urdf (robot description, URDF)
Before this commit: robot tree.urdf, 1 links, 0 joints
Links:
- link baseLink: geometry collision mesh filename=real_tree2.obj scale=1 1 1; visual mesh filename=real_tree2.stl scale=1 1 1

Commit message: Failed attempt at capturing the in-hand point cloud. Working on cloning approach angles.

File: data/real_tree.urdf (robot description, URDF)
Before this commit: robot tree.urdf, 1 links, 0 joints
Links:
- link baseLink: geometry collision mesh filename=real_tree2.obj scale=1 1 1; visual mesh filename=real_tree2.obj scale=1 1 1
