Commit message: Convex decomposition of gripper fingers. Use pick contact points and not nearby points. New demos.

File: data/robotiq.urdf (robot description, URDF)
Before this commit: robot robotiq_85_gripper, 9 links, 8 joints
Links:
- link robotiq_85_left_finger_tip_link: geometry collision mesh filename=robotiq_description/meshes/collision/robotiq_85_finger_link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; visual mesh filename=robotiq_description/meshes/visual/robotiq_85_finger_tip_lin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
- link robotiq_85_right_finger_tip_link: geometry collision mesh filename=robotiq_description/meshes/collision/robotiq_85_finger_link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; visual mesh filename=robotiq_description/meshes/visual/robotiq_85_finger_tip_lin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
